File: Nya RT-datorn/CÅ-815/Schema/CÅ-815.kicad_sch (KiCad schematic)
At the start: 57 parts, among them IC1 RT-74LS245, IC10 6821, IC11 6116, IC12 74LS374, IC13 MCM66790, IC14 555, IC15 555, IC16 74LS30, IC17 74LS02, IC18 DM8602, IC19 74LS74, IC2 RT-74LS245, IC20 74LS00, IC21 74LS74, IC22 74LS02, IC23 74LS165, IC24 74LS86, IC25 74LS06, IC3 MC6845, IC4 74LS157, IC5 74LS157, IC6 74LS157, IC7 74LS04, IC8 74LS163, IC9 74LS174, J1 Tangentbordskontakt, P1 C64AC, T1 BC378, X1 16MHz

Commit message: Uppdaterade CÅ-815
Parts:
- D1: value D -> 1N4148
- IC1, IC2: symbol RT-lib:RT-74LS245 -> CÅ-815:RT-74LS245
- IC10: symbol RT-lib:RT-6821 -> CÅ-815:RT-6821
- IC11: symbol RT-lib:6116 -> CÅ-815:6116
- IC12: symbol RT-lib:RT-74LS374 -> CÅ-815:RT-74LS374
- IC13: symbol RT-lib:MCM66790 -> CÅ-815:MCM66790
- IC18: symbol RT-lib:DM8602 -> CÅ-815:DM8602
- IC19, IC21: symbol RT-lib:RT-74LS74 -> CÅ-815:RT-74LS74
- IC23: symbol RT-lib:RT-74LS165 -> CÅ-815:RT-74LS165
- IC3: symbol RT-lib:RT-MC6845 -> CÅ-815:RT-MC6845
- IC4, IC5, IC6: symbol RT-lib:RT-74LS157 -> CÅ-815:RT-74LS157
- IC8: symbol RT-lib:74LS163 -> CÅ-815:74LS163
- IC9: symbol RT-lib:RT-74LS174 -> CÅ-815:RT-74LS174
- J1: symbol RT-lib:Conn_01x26 -> CÅ-815:Conn_01x26
- P1: value C64AC -> RT-bus; symbol RT-lib:C64AC -> CÅ-815:RT-bus
Changed lines of the file:
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@@
   (title_block
     (title "CÅ-815 CRTC")
-    (date "2023-07-11")
-    (rev "0.99")
+    (date "2023-07-30")
+    (rev "1.0")
     (company "Åke Holm, CÅ-Elektronik")
     (comment 1 "Nya RT-datorn")
     (comment 2 "Videoterminal baserad på 6845")
+    (comment 3 "Schema skapat av Mikael karlsson")
   )
   (junction (at 286.385 299.085) (diameter 0) (color 0 0 0 0)
@@
     (stroke (width 0) (type default))
   )
+  (wire (pts (xy 285.115 212.09) (xy 283.845 212.09))
+    (stroke (width 0) (type default))
+  )
   (wire (pts (xy 82.55 104.775) (xy 85.09 104.775))
     (stroke (width 0) (type default))
@@
     )
   )
-  (symbol (lib_id "RT-lib:RT-74LS74") (at 99.695 368.3 0) (unit 3)
+  (symbol (lib_id "CÅ-815:RT-74LS74") (at 99.695 368.3 0) (unit 3)
     (in_bom yes) (on_board yes) (dnp no)
     (property "Reference" "IC21" (at 96.901 367.03 0)
@@
     )
   )
-  (symbol (lib_id "RT-lib:RT-74LS245") (at 253.365 92.71 0) (unit 1)
+  (symbol (lib_id "CÅ-815:RT-74LS245") (at 253.365 92.71 0) (unit 1)
     (in_bom yes) (on_board yes) (dnp no)
     (property "Reference" "IC2" (at 253.365 90.17 0)
@@
     )
   )
-  (symbol (lib_id "RT-lib:RT-74LS157") (at 240.665 162.56 0) (unit 1)
+  (symbol (lib_id "CÅ-815:RT-74LS157") (at 240.665 162.56 0) (unit 1)
     (in_bom yes) (on_board yes) (dnp no)
     (property "Reference" "IC4" (at 241.3 161.925 0)
@@
     )
   )
-  (symbol (lib_id "RT-lib:RT-74LS245") (at 184.785 92.71 0) (unit 1)
+  (symbol (lib_id "CÅ-815:RT-74LS245") (at 184.785 92.71 0) (unit 1)
     (in_bom yes) (on_board yes) (dnp no)
     (property "Reference" "IC1" (at 184.15 90.805 0)
@@
     )
   )
-  (symbol (lib_id "RT-lib:RT-74LS74") (at 78.105 368.3 0) (unit 3)
+  (symbol (lib_id "CÅ-815:RT-74LS74") (at 78.105 368.3 0) (unit 3)
     (in_bom yes) (on_board yes) (dnp no)
     (property "Reference" "IC19" (at 75.311 367.03 0)
@@
     )
   )
+  (symbol (lib_id "power:+5V") (at 285.115 212.09 270) (unit 1)
+    (in_bom yes) (on_board yes) (dnp no) (fields_autoplaced)
+    (property "Reference" "#PWR039" (at 281.305 212.09 0)
+      (effects (font (size 1.27 1.27)) hide)
+    )
+    (property "Value" "+5V" (at 288.29 212.09 90)
+      (effects (font (size 1.27 1.27)) (justify left) hide)
+    )
+    (property "Footprint" "" (at 285.115 212.09 0)
+      (effects (font (size 1.27 1.27)) hide)
+    )
+    (property "Datasheet" "" (at 285.115 212.09 0)
+      (effects (font (size 1.27 1.27)) hide)
+    )
+    (pin "1")
+    (instances
+      (project "CÅ-815"
+        (path "/b61304a0-6813-46ba-9781-62901ee88403"
+          (reference "#PWR039") (unit 1)
+        )
+      )
+    )
+  )
   (symbol (lib_id "Device:R") (at 171.45 337.82 0) (unit 1)
     (in_bom yes) (on_board yes) (dnp no)
@@
     )
   )
-  (symbol (lib_id "RT-lib:RT-74LS74") (at 348.615 244.475 0) (unit 2)
+  (symbol (lib_id "CÅ-815:RT-74LS74") (at 348.615 244.475 0) (unit 2)
     (in_bom yes) (on_board yes) (dnp no)
     (property "Reference" "IC19" (at 346.075 243.062 0)
@@
     )
   )
-  (symbol (lib_id "RT-lib:RT-6821") (at 414.655 92.71 0) (unit 1)
+  (symbol (lib_id "CÅ-815:RT-6821") (at 414.655 92.71 0) (unit 1)
     (in_bom yes) (on_board yes) (dnp no)
     (property "Reference" "IC10" (at 415.29 91.44 0)
@@
     )
   )
-  (symbol (lib_id "power:+5V") (at 283.845 212.09 270) (unit 1)
-    (in_bom yes) (on_board yes) (dnp no) (fields_autoplaced)
-    (property "Reference" "#PWR039" (at 280.035 212.09 0)
-      (effects (font (size 1.27 1.27)) hide)
-    )
-    (property "Value" "+5V" (at 287.02 212.09 90)
-      (effects (font (size 1.27 1.27)) (justify left) hide)
-    )
-    (property "Footprint" "" (at 283.845 212.09 0)
-      (effects (font (size 1.27 1.27)) hide)
-    )
-    (property "Datasheet" "" (at 283.845 212.09 0)
-      (effects (font (size 1.27 1.27)) hide)
-    )
-    (pin "1")
-    (instances
-      (project "CÅ-815"
-        (path "/b61304a0-6813-46ba-9781-62901ee88403"
-          (reference "#PWR039") (unit 1)
-        )
-      )
-    )
-  )
   (symbol (lib_id "74xx:74LS86") (at 369.57 312.42 0) (mirror x) (unit 3)
     (in_bom yes) (on_board yes) (dnp no)
@@
     )
   )
-  (symbol (lib_name "DM8602_2") (lib_id "RT-lib:DM8602") (at 189.865 349.25 0) (unit 1)
+  (symbol (lib_name "DM8602_2") (lib_id "CÅ-815:DM8602") (at 189.865 349.25 0) (unit 1)
     (in_bom yes) (on_board yes) (dnp no) (fields_autoplaced)
     (property "Reference" "IC18" (at 189.865 338.05 0)
@@
   (symbol (lib_id "Device:D") (at 267.335 325.12 0) (unit 1)
     (in_bom yes) (on_board yes) (dnp no) (fields_autoplaced)
-    (property "Reference" "D1" (at 267.335 320.27 0)
+    (property "Reference" "D1" (at 267.335 319.7057 0)
       (effects (font (size 1.27 1.27)))
     )
-    (property "Value" "D" (at 267.335 322.318 0)
+    (property "Value" "1N4148" (at 267.335 322.1299 0)
       (effects (font (size 1.27 1.27)))
     )
@@
     )
   )
-  (symbol (lib_id "RT-lib:RT-74LS374") (at 327.025 132.715 0) (unit 1)
+  (symbol (lib_id "CÅ-815:RT-74LS374") (at 327.025 132.715 0) (unit 1)
     (in_bom yes) (on_board yes) (dnp no)
     (property "Reference" "IC12" (at 327.025 131.302 0)
@@
     )
   )
-  (symbol (lib_id "RT-lib:DM8602") (at 189.865 306.705 0) (unit 2)
+  (symbol (lib_id "CÅ-815:DM8602") (at 189.865 306.705 0) (unit 2)
     (in_bom yes) (on_board yes) (dnp no) (fields_autoplaced)
     (property "Reference" "IC18" (at 189.865 295.505 0)
@@
     )
   )
-  (symbol (lib_id "RT-lib:RT-74LS157") (at 258.445 185.42 0) (unit 1)
+  (symbol (lib_id "CÅ-815:RT-74LS157") (at 258.445 185.42 0) (unit 1)
     (in_bom yes) (on_board yes) (dnp no)
     (property "Reference" "IC5" (at 258.445 184.785 0)
@@
     )
   )
-  (symbol (lib_id "RT-lib:6116") (at 253.365 133.985 0) (unit 1)
+  (symbol (lib_id "CÅ-815:6116") (at 253.365 133.985 0) (unit 1)
     (in_bom yes) (on_board yes) (dnp no)
     (property "Reference" "IC11" (at 253.365 133.307 0)
@@
     )
   )
-  (symbol (lib_id "RT-lib:RT-74LS74") (at 213.995 325.12 0) (unit 1)
+  (symbol (lib_id "CÅ-815:RT-74LS74") (at 213.995 325.12 0) (unit 1)
     (in_bom yes) (on_board yes) (dnp no) (fields_autoplaced)
     (property "Reference" "IC19" (at 215.9509 316.46 0)
@@
     )
   )
-  (symbol (lib_id "RT-lib:RT-74LS157") (at 276.225 208.28 0) (unit 1)
+  (symbol (lib_id "CÅ-815:RT-74LS157") (at 276.225 208.28 0) (unit 1)
     (in_bom yes) (on_board yes) (dnp no)
     (property "Reference" "IC6" (at 276.225 208.28 0)
@@
     )
   )
-  (symbol (lib_id "RT-lib:RT-MC6845") (at 184.785 171.45 0) (unit 1)
+  (symbol (lib_id "CÅ-815:RT-MC6845") (at 184.785 171.45 0) (unit 1)
     (in_bom yes) (on_board yes) (dnp no)
     (property "Reference" "IC3" (at 182.88 170.815 0)
@@
     )
   )
-  (symbol (lib_id "RT-lib:RT-74LS74") (at 396.24 251.46 0) (unit 2)
+  (symbol (lib_id "CÅ-815:RT-74LS74") (at 396.24 251.46 0) (unit 2)
     (in_bom yes) (on_board yes) (dnp no) (fields_autoplaced)
     (property "Reference" "IC21" (at 398.1959 242.8 0)
@@
     )
   )
-  (symbol (lib_id "RT-lib:C64AC") (at 69.85 174.625 180) (unit 1)
+  (symbol (lib_id "CÅ-815:RT-bus") (at 69.85 174.625 180) (unit 1)
     (in_bom yes) (on_board yes) (dnp no) (fields_autoplaced)
     (property "Reference" "P1" (at 68.58 88.622 0)
       (effects (font (size 1.27 1.27)))
     )
-    (property "Value" "C64AC" (at 68.58 90.67 0)
+    (property "Value" "RT-bus" (at 68.58 90.67 0)
       (effects (font (size 1.27 1.27)))
     )
@@
     )
   )
-  (symbol (lib_id "RT-lib:RT-74LS174") (at 224.79 259.08 0) (unit 1)
+  (symbol (lib_id "CÅ-815:RT-74LS174") (at 224.79 259.08 0) (unit 1)
     (in_bom yes) (on_board yes) (dnp no)
     (property "Reference" "IC9" (at 224.79 257.175 0)
@@
     )
   )
-  (symbol (lib_id "RT-lib:74LS163") (at 336.55 269.875 0) (unit 1)
+  (symbol (lib_id "CÅ-815:74LS163") (at 336.55 269.875 0) (unit 1)
     (in_bom yes) (on_board yes) (dnp no)
     (property "Reference" "IC8" (at 336.55 268.605 0)
@@
     )
   )
-  (symbol (lib_id "RT-lib:Conn_01x26") (at 488.95 168.91 0) (unit 1)
+  (symbol (lib_id "CÅ-815:Conn_01x26") (at 488.95 168.91 0) (unit 1)
     (in_bom yes) (on_board yes) (dnp no)
     (property "Reference" "J1" (at 490.855 135.89 0)
@@
     )
   )
-  (symbol (lib_id "RT-lib:MCM66790") (at 325.755 161.29 0) (unit 1)
+  (symbol (lib_id "CÅ-815:MCM66790") (at 325.755 161.29 0) (unit 1)
     (in_bom yes) (on_board yes) (dnp no)
     (property "Reference" "IC13" (at 325.755 159.385 0)
@@
     )
   )
-  (symbol (lib_name "DM8602_1") (lib_id "RT-lib:DM8602") (at 67.31 368.3 0) (unit 3)
+  (symbol (lib_name "DM8602_1") (lib_id "CÅ-815:DM8602") (at 67.31 368.3 0) (unit 3)
     (in_bom yes) (on_board yes) (dnp no)
-    (property "Reference" "IC18" (at 64.77 367.395 0)
+    (property "Reference" "IC18" (at 63.5 367.03 0)
       (effects (font (size 1.27 1.27)) (justify left))
     )
-    (property "Value" "DM8602" (at 64.77 369.443 0)
+    (property "Value" "DM8602" (at 63.5 369.078 0)
       (effects (font (size 1.27 1.27)) (justify left))
     )
@@
     )
   )
-  (symbol (lib_id "RT-lib:RT-74LS165") (at 325.755 189.865 0) (unit 1)
+  (symbol (lib_id "CÅ-815:RT-74LS165") (at 325.755 189.865 0) (unit 1)
     (in_bom yes) (on_board yes) (dnp no)
     (property "Reference" "IC23" (at 330.835 187.817 0)
@@
     )
   )
-  (symbol (lib_id "RT-lib:RT-74LS74") (at 396.24 280.035 270) (mirror x) (unit 1)
+  (symbol (lib_id "CÅ-815:RT-74LS74") (at 396.24 280.035 270) (mirror x) (unit 1)
     (in_bom yes) (on_board yes) (dnp no)
     (property "Reference" "IC21" (at 407.035 284.48 90)

Commit message: Updated RT-bus connector on all schematics
Parts:
- R2: value R -> 4.7k
Connections:
- net +5V: now also P1.a30 (+5V), P1.a31 (+5V), P1.a32 (+5V), P1.c30 (+5V), P1.c31 (+5V), P1.c32 (+5V); no longer P1.30A (+5V), P1.30C (+5V), P1.31A (+5V), P1.31C (+5V), P1.32A (+5V), P1.32C (+5V)
- net A0: now also P1.a18 (A0); no longer P1.18A (A0)
- net A1: now also P1.c18 (A1); no longer P1.18C (A1)
- net A10: now also P1.a13 (A10); no longer P1.13A (A10)
- net A2: now also P1.a17 (A2); no longer P1.17A (A2)
- net A3: now also P1.c17 (A3); no longer P1.17C (A3)
- net A4: now also P1.a16 (A4); no longer P1.16A (A4)
- net A5: now also P1.c16 (A5); no longer P1.16C (A5)
- net A6: now also P1.a15 (A6); no longer P1.15A (A6)
- net A7: now also P1.c15 (A7); no longer P1.15C (A7)
- net A8: now also P1.a14 (A8); no longer P1.14A (A8)
- net A9: now also P1.c14 (A9); no longer P1.14C (A9)
- net BD0: now also P1.c22 (D0); no longer P1.22C (D0)
- net BD1: now also P1.c23 (D1); no longer P1.23C (D1)
- net BD2: now also P1.c24 (D2); no longer P1.24C (D2)
- net BD3: now also P1.c25 (D3); no longer P1.25C (D3)
- net BD4: now also P1.c26 (D4); no longer P1.26C (D4)
- net BD5: now also P1.c27 (D5); no longer P1.27C (D5)
- net BD6: now also P1.c28 (D6); no longer P1.28C (D6)
- net BD7: now also P1.c29 (D7); no longer P1.29C (D7)
- net GND: now also P1.a1 (GND), P1.a2 (GND), P1.a22 (GND), P1.a23 (GND), P1.a24 (GND), P1.a25 (GND), P1.a26 (GND), P1.a27 (GND), P1.a28 (GND), P1.a29 (GND), P1.a3 (GND), P1.c1 (GND), P1.c2 (GND), P1.c21 (GND), P1.c3 (GND); no longer P1.1A (GND), P1.1C (GNC), P1.21C (GND), P1.22A (GND), P1.23A (GND), P1.24A (GND), P1.25A (GND), P1.26A (GND), P1.27A (GND), P1.28A (GND), P1.29A (GND), P1.2A (GND), P1.2C (GND), P1.3A (GND), P1.3C (GND)
- net ID0: now also IC11.17 (Q7), IC12.18 (D7), IC2.2 (A0); no longer IC11.16 (Q6), IC12.3 (D0), IC2.9 (A7)
- net ID1: now also IC11.13 (Q3), IC12.8 (D3), IC2.3 (A1); no longer IC11.9 (Q0), IC12.4 (D1), IC2.8 (A6)
- net ID2: now also IC11.11 (Q2), IC12.13 (D4), IC2.4 (A2); no longer IC11.15 (Q5), IC12.17 (D6), IC2.7 (A5)
- net ID3: now also IC11.14 (Q4), IC12.7 (D2), IC2.5 (A3); no longer IC11.10 (Q1), IC12.14 (D5), IC2.6 (A4)
- net ID4: now also IC11.10 (Q1), IC12.14 (D5), IC2.6 (A4); no longer IC11.14 (Q4), IC12.7 (D2), IC2.5 (A3)
- net ID5: now also IC11.15 (Q5), IC12.17 (D6), IC2.7 (A5); no longer IC11.11 (Q2), IC12.13 (D4), IC2.4 (A2)
- net ID6: now also IC11.9 (Q0), IC12.4 (D1), IC2.8 (A6); no longer IC11.13 (Q3), IC12.8 (D3), IC2.3 (A1)
- net ID7: now also IC11.16 (Q6), IC12.3 (D0), IC2.9 (A7); no longer IC11.17 (Q7), IC12.18 (D7), IC2.2 (A0)
- net at IC1.1 (A->B), IC10.21 (R/~{W}), IC2.1 (A->B)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: now also P1.c19 (R/~{W}); no longer P1.19C (R/W)
- net at IC2.19 (CE), IC21.13 (~{R}), IC22.8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: now also P1.c10 (~{E800}); no longer P1.10C (E800)
- net at IC10.25 (ENABLE), IC20.13, IC3.23 (E): now also P1.c20 (E); no longer P1.20C (E)
- net at IC10.34 (~{RESET}), IC3.2 (~{RESET}): now also P1.a20 (RESET); no longer P1.20A (RESET)
- net at IC17.5: now also P1.a19 (I/O-Select); no longer P1.19A (I/O-Select)
Other:
- moved on the sheet: IC7E
